Commit message: rotated such that x is forward

File: rover_desc/parts/robot.urdf (robot description, URDF)
Before this commit: robot rover, 29 links, 28 joints
Links:
- removed link rover_base
- added link base_link
Joints:
- removed joint base_link_to_base
- added joint base_link_to_body: type fixed, parent base_link, child body, origin xyz=0 0 0 rpy=0.0 0 +1.570796

File: rover_desc/rover.xacro (robot description, xacro)
@@ -3,15 +3,3 @@
     <!-- URDF & Visual -->
     <xacro:include filename="$(find rover_description)/rover_desc/parts/robot.urdf" />
-    <xacro:include filename="$(find rover_description)/rover_desc/gazebo_params.xacro" />
-    <xacro:include filename="$(find rover_description)/rover_desc/realsense.urdf" />
-    <xacro:include filename="$(find rover_description)/rover_desc/gz_realsense.xacro"/>
-    <xacro:realsense_d435 parent="imager_3">
-        <origin xyz="-0.0325 0 -0.005" rpy="${pi/2} ${pi/2} ${0}"/>
-    </xacro:realsense_d435>
-    <!-- Include ros2_control -->
-    <xacro:include filename="$(find rover_gz)/plugins/ros2_control.xacro" />
-    <xacro:include filename="$(find rover_description)/rover_desc/imu.xacro" />
-    <xacro:imu_sensor parent="rover_base">
-        <origin xyz="0.28136771400569077217 -0.651070713998295858 0.42390609907984444504" rpy="0 0 0"/>
-    </xacro:imu_sensor>
 </robot>

Commit message: pleasepelase

File: rover_desc/parts/robot.urdf (robot description, URDF)
Before this commit: robot rover, 29 links, 28 joints
Joints:
- joint base_link_to_body: origin xyz=0 0 0 rpy=0.0 0 +1.570796 -> xyz=0 0 0 rpy=0 0 1.5707963267948952257

File: rover_desc/realsense.urdf (robot description, URDF)
Before this commit: robot rover, 10 links, 10 joints
Links:
- added link realsense_link
- link camera_link: geometry collision mesh filename=file://$(find realsense2_description)/meshes/d435.dae; visual mesh filename=file://$(find realsense2_description)/meshes/d435.dae
Joints:
- added joint realsense_joint: type fixed, parent yaw, child realsense_link

File: rover_desc/rover.xacro (robot description, xacro)
@@ -2,4 +2,22 @@
 <robot xmlns:xacro="http://ros.org/wiki/xacro" name="rover">
     <!-- URDF & Visual -->
-    <xacro:include filename="$(find rover_description)/rover_desc/parts/robot.urdf" />
+    <!-- <xacro:include filename="$(find rover_description)/rover_desc/realsense.urdf" /> -->
+    <xacro:include filename="$(find rover_description)/rover_desc/_d435.urdf.xacro" />
+    <link name="base_link">
+    </link>
+    <xacro:sensor_d435
+        parent="base_link"
+        name="camera"
+        use_nominal_extrinsics="true"
+        add_plug="false"
+        use_mesh="true">
+        <origin xyz="0.47136771400569088541 -0.60607071399829648417 0.26237109907984434987" rpy="0 0 0"/>
+    </xacro:sensor_d435>
+    <!-- <xacro:include filename="$(find rover_description)/rover_desc/parts/robot.urdf" /> -->
+    <!-- <link name="camera_link"></link>
+    <joint name="camera_link_joint" type="fixed">
+        <parent link="rs_pitch" />
+        <child link="camera_link" />
+        <origin xyz="0 0 0.1 " rpy="0 0 0" />
+    </joint> -->
 </robot>
