Commit message: autonomy

File: rover_desc/rover.xacro (robot description, xacro)
@@ -14,4 +14,10 @@
         <origin xyz="0.47136771400569088541 -0.60607071399829648417 0.26237109907984434987" rpy="0 0 0"/>
     </xacro:sensor_d435>
+    <joint name="laser_joint" type="fixed">
+        <parent link="base_link"/>
+        <child link="laser"/>
+        <origin xyz="0 0 0.15" rpy="0 0 0"/>
+    </joint>
+    <link name="laser"/>
     <!-- <xacro:include filename="$(find rover_description)/rover_desc/parts/robot.urdf" /> -->
     <!-- <link name="camera_link"></link>

Commit message: reverting to simplier

File: rover_desc/rover.xacro (robot description, xacro)
@@ -12,12 +12,12 @@
         add_plug="false"
         use_mesh="true">
-        <origin xyz="0.47136771400569088541 -0.60607071399829648417 0.26237109907984434987" rpy="0 0 0"/>
+        <origin xyz="0.0 0.0 0.0" rpy="0 0 0"/>
     </xacro:sensor_d435>
-    <joint name="laser_joint" type="fixed">
+    <!-- <joint name="laser_joint" type="fixed">
         <parent link="base_link"/>
         <child link="laser"/>
-        <origin xyz="0 0 0.15" rpy="0 0 0"/>
+        <origin xyz="0 0 0.0" rpy="0 0 0"/>
     </joint>
-    <link name="laser"/>
+    <link name="laser"/> -->
     <!-- <xacro:include filename="$(find rover_description)/rover_desc/parts/robot.urdf" /> -->
     <!-- <link name="camera_link"></link>
